Commit message: Add mm_navigation package and clean up mm_description
- Remove ros2_control remnants (omni_kinematics.cpp, ros2_control xacro,
  wheel xacro, ros2_controllers yaml) — replaced by Gazebo plugin baseline
- Add cmd_vel_smoother.py and custom_keyboard_control.py scripts
- Update gazebo.launch.py to start cmd_vel_smoother node
- Update display_model.rviz with Map display (Transient Local QoS) and nav tools
- Add mm_navigation package: nav2_params.yaml (tuned for 400mm omni base),
  navigation2.launch.py, and room map (pgm + yaml)

File: mm_description/urdf/omni_base.urdf.xacro (robot description, xacro)
@@ -11,7 +11,7 @@
     <color rgba="0.9 0.1 0.1 1.0"/>
   </material>
-  <!-- 底盘参数 - 400mm x 400mm -->
-  <xacro:property name="body_length" value="0.40"/>
-  <xacro:property name="body_width" value="0.40"/>
+  <!-- 底盘参数 - 整车投影约 400mm x 400mm -->
+  <xacro:property name="body_length" value="0.30"/>
+  <xacro:property name="body_width" value="0.30"/>
   <xacro:property name="body_height" value="0.03"/>
   <!-- 轮子参数 -->
@@ -41,7 +41,7 @@
   <link name="base_footprint"/>
   <joint name="base_footprint_joint" type="fixed">
-    <parent link="base_link"/>
-    <child link="base_footprint"/>
-    <origin xyz="0 0 -${wheel_radius}" rpy="0 0 0"/>
+    <parent link="base_footprint"/>
+    <child link="base_link"/>
+    <origin xyz="0 0 ${wheel_radius}" rpy="0 0 0"/>
   </joint>
   <!-- 激光雷达链接 -->
@@ -52,4 +52,11 @@
       </geometry>
       <material name="red"/>
+    </visual>
+    <visual>
+      <origin xyz="-0.035 0 0.015" rpy="0 0 0"/>
+      <geometry>
+        <box size="0.025 0.09 0.03"/>
+      </geometry>
+      <material name="black"/>
     </visual>
     <collision>
@@ -196,6 +203,6 @@
             <samples>720</samples>
             <resolution>1</resolution>
-            <min_angle>-3.14159</min_angle>
-            <max_angle>3.14159</max_angle>
+            <min_angle>-2.35619</min_angle>
+            <max_angle>2.35619</max_angle>
           </horizontal>
         </scan>
@@ -218,5 +225,5 @@
   <gazebo>
     <plugin name="object_controller" filename="libgazebo_ros_planar_move.so">
-      <commandTopic>cmd_vel</commandTopic>
+      <commandTopic>cmd_vel_smoothed</commandTopic>
       <odometryTopic>odom</odometryTopic>
       <odometryFrame>odom</odometryFrame>

Commit message: Update navigation and simulation setup

File: mm_description/urdf/omni_base.urdf.xacro (robot description, xacro)
@@ -53,11 +53,4 @@
       <material name="red"/>
     </visual>
-    <visual>
-      <origin xyz="-0.035 0 0.015" rpy="0 0 0"/>
-      <geometry>
-        <box size="0.025 0.09 0.03"/>
-      </geometry>
-      <material name="black"/>
-    </visual>
     <collision>
       <geometry>
@@ -197,19 +190,24 @@
       <pose>0 0 0 0 0 0</pose>
       <visualize>true</visualize>
-      <update_rate>15</update_rate>
+      <update_rate>10</update_rate>
       <ray>
         <scan>
           <horizontal>
-            <samples>720</samples>
+            <samples>1200</samples>
             <resolution>1</resolution>
-            <min_angle>-2.35619</min_angle>
-            <max_angle>2.35619</max_angle>
+            <min_angle>-2.61799</min_angle>
+            <max_angle>2.61799</max_angle>
           </horizontal>
         </scan>
         <range>
           <min>0.12</min>
-          <max>12.0</max>
+          <max>25.0</max>
           <resolution>0.01</resolution>
         </range>
+        <noise>
+          <type>gaussian</type>
+          <mean>0.0</mean>
+          <stddev>0.01</stddev>
+        </noise>
       </ray>
       <plugin name="laser_plugin" filename="libgazebo_ros_ray_sensor.so">
@@ -225,5 +223,5 @@
   <gazebo>
     <plugin name="object_controller" filename="libgazebo_ros_planar_move.so">
-      <commandTopic>cmd_vel_smoothed</commandTopic>
+      <commandTopic>cmd_vel</commandTopic>
       <odometryTopic>odom</odometryTopic>
       <odometryFrame>odom</odometryFrame>
