Commit message: sim 1 "nav and moveit"

File: mm_description/urdf/mm_robot.urdf (robot description, URDF)
Before this commit: robot robot, 17 links, 16 joints
Joints:
- joint Joint_1: axis 0 0 1 -> (none); type continuous -> fixed
- joint Joint_2: axis 0 0 1 -> (none); type continuous -> fixed
- joint Joint_3: axis 0 0 1 -> (none); type continuous -> fixed
- joint Joint_4: axis 0 0 1 -> (none); type continuous -> fixed
