Commit message: docs更新

File: mm_description/urdf/mm_robot.urdf (robot description, URDF)
Before this commit: robot robot, 17 links, 16 joints
Links:
- added link suction_link, mass 0.02; collision cylinder length=0.03 radius=0.0075; visual cylinder length=0.03 radius=0.0075
- added link suction_tip
Joints:
- added joint Joint_suction: type fixed, parent Link_29, child suction_link, origin xyz=0 0 0 rpy=0 0 0
- added joint Joint_suction_tip: type fixed, parent suction_link, child suction_tip, origin xyz=0 0 -0.095 rpy=0 0 0

Commit message: 机械臂零位更新

File: mm_description/urdf/mm_robot.urdf (robot description, URDF)
Before this commit: robot robot, 19 links, 18 joints
Joints:
- joint Joint_11: axis 0 0 -1 -> 0 0 1; limit lower=0 upper=4.712 effort=10 velocity=1 -> lower=0 upper=4.74690659 effort=10 velocity=1; origin xyz=0 0 0.0974 rpy=0 0 -2.38237443 -> xyz=0 0 0.0974 rpy=0 0 -0.84609571
- joint Joint_16: axis 0 0 1 -> 0 0 -1; limit lower=-1.571 upper=1.571 effort=10 velocity=1 -> lower=0 upper=5.55014702 effort=10 velocity=1; origin xyz=5e-8 -0.046 -0.0251 rpy=1.57079633 0.00872784 3.14159265 -> xyz=5e-8 -0.046 -0.0251 rpy=-1.57079633 -0.28798052 0

Commit message: 零位调整

File: mm_description/urdf/mm_robot.urdf (robot description, URDF)
Before this commit: robot robot, 19 links, 18 joints
Joints:
- joint Joint_11: limit lower=0 upper=4.74690659 effort=10 velocity=1 -> lower=0 upper=4.7469066 effort=10 velocity=1; origin xyz=0 0 0.0974 rpy=0 0 -0.84609571 -> xyz=0 0 0.0974 rpy=0 0 -0.84609572
- joint Joint_16: origin xyz=5e-8 -0.046 -0.0251 rpy=-1.57079633 -0.28798052 0 -> xyz=5e-8 -0.046 -0.0251 rpy=-1.57079633 -0.21816735 0

Commit message: j6零位调整

File: mm_description/urdf/mm_robot.urdf (robot description, URDF)
Before this commit: robot robot, 19 links, 18 joints
Joints:
- joint Joint_16: origin xyz=5e-8 -0.046 -0.0251 rpy=-1.57079633 -0.21816735 0 -> xyz=5e-8 -0.046 -0.0251 rpy=-1.57079633 -0.18326076 0

Commit message: fix(description,navigation): 新增 laser_link 测量帧修雷达手性 + 自遮挡滤除 + 建图配置
雷达"前后颠倒"真机实测定案(挡测法, 每次 100 帧取最小):
  挡车头(base 0°) -> scan 报 180°;  挡车左(base +90°) -> scan 报 -90°
唯一解 theta_scan = theta_base + 180, 即纯旋转无镜像(镜像假设预测挡左出现在
+90°, 已被实测排除)。而旧 URDF Joint_6 的 roll=-pi 让下游算出
theta_base = -theta_scan: 左右对、前后反。仿真里看不出是因为 Gazebo 在同一个
翻转帧里生成射线, 自洽 —— 这个偏差因此藏了两个月。

不直接改 Joint_6 的 rpy, 而是新增 laser_link: Link_12.stl 主体画在自身坐标系
Z 负半侧, roll=-pi 是 mesh 需要的; 改 yaw=pi 则 mesh 陷进底盘, 而 Link_12 带
collision 供 MoveIt 自碰撞检查用, 雷达碰撞体位置错了会让臂扫过雷达真实位置时
不报碰撞。一个帧满足不了 mesh(Rx) 与 scan(Rz) 两个需求, 故拆开。

配套: 仿真 sensor 射线改在 laser_link 生成(pose pitch=pi), FOV 300°->360°
(真机 A3 本就发 360°, 后方遮挡交 laser_filters 统一处理, 两边同一个 filter);
新增 scan_filter 砍臂自遮挡扇区(ready 姿态实测只 base 160~180°, 取 ±25° 留
近一倍余量, 保住 310° 视野); slam_toolbox 建图配置与 mapping.launch.py。

顺手修一个真 bug: EKF 硬编码发 /odometry/filtered, 而 nav2_params 里
controller_server 与 velocity_smoother 都订 /odom 且两边都没 remap ->
Nav2 拿不到里程计, 表现是控制器不出 cmd_vel 却不报错。

ekf.yaml 关掉 imu0 的 vyaw 位: 实测固件发的 angular_velocity 三轴恒为 0
(静止 383 帧一个 bit 不变), 开着等于持续告诉 EKF "车没在转", 与 odom0 的真实
vyaw 观测冲突。固件补上后可改回 true。

File: mm_description/urdf/mm_robot.urdf (robot description, URDF)
Before this commit: robot robot, 19 links, 18 joints
Links:
- added link laser_link
Joints:
- added joint Joint_laser: type fixed, parent base_link, child laser_link, origin xyz=0.10568947 -0.00001261 0.22079956 rpy=0 0 3.14159265

File: mm_description/urdf/mm_robot_gazebo.urdf.xacro (robot description, xacro)
@@ -78,10 +78,16 @@
     <xacro:wheel_frictionless link="Link_9"/>
     <xacro:wheel_frictionless link="Link_10"/>
-    <!-- 雷达 sensor: 挂在整车雷达 link (Link_12). Link_12 在 base_link 中 X=前/Y=右/Z=下,
-         扫描平面水平、0°对准车头; Z 朝下只影响角度手性, frame_id=Link_12 + TF 自洽.
-         ±150°(总300°) 盲区落在车后. (参数移植自旧 omni_base.urdf.xacro) -->
+    <!-- 雷达 sensor: 射线在 **laser_link**(测量帧) 里生成, 与真机驱动一致.
+         2026-08-08 改: 原先射线在 Link_12(mesh 帧) 里生成、frame_name=Link_12, 仿真内部自洽,
+         但真机雷达实际绕竖轴转了 180° 装 —— 于是 sim 对 real 错, 这个偏差藏了两个月.
+         现在两边共用同一个测量帧定义 (laser_link, 见 mm_robot.urdf 的 Joint_laser).
+         sensor 仍挂 Link_12(gazebo 的 reference 要求是带惯量的真 link), 靠 pose 把射线
+         转到 laser_link 朝向: Rx(pi)^-1 · Rz(pi) = Ry(pi), 故 pitch=pi.
+         FOV 改 360°(原 ±150°): 真机 A3 驱动本来就发完整 360°, 仿真砍成 300° 是不真实的.
+         "后方看不见"的真正来源是机械臂遮挡 —— 那由 laser_filters 砍扇区统一处理
+         (sim 里 URDF 已有臂几何, Gazebo 射线会自然自遮挡, 再过同一个 filter 就与真机一致). -->
     <gazebo reference="Link_12">
         <sensor name="lidar_sensor" type="ray">
-            <pose>0 0 0 0 0 0</pose>
+            <pose>0 0 0 0 3.14159265 0</pose>
             <visualize>true</visualize>
             <update_rate>10</update_rate>
@@ -89,8 +95,8 @@
                 <scan>
                     <horizontal>
-                        <samples>1200</samples>
+                        <samples>720</samples>
                         <resolution>1</resolution>
-                        <min_angle>-2.61799</min_angle>
-                        <max_angle>2.61799</max_angle>
+                        <min_angle>-3.14159265</min_angle>
+                        <max_angle>3.14159265</max_angle>
                     </horizontal>
                 </scan>
@@ -111,5 +117,5 @@
                 </ros>
                 <output_type>sensor_msgs/LaserScan</output_type>
-                <frame_name>Link_12</frame_name>
+                <frame_name>laser_link</frame_name>
             </plugin>
         </sensor>
