Commit message: feat(sim): M4/M5 抓取节点 + 任务状态机 + 导航回报
- mm_grasp: grasp_node 三段抓取 + /grasp/execute /grasp/unload
- mm_task: mission_manager S0-S5 状态机 + mission.yaml
- lane_navigator: 加 /lane_navigator/status 导航回报
- mock_suction 假吸附 + place_box_helper 摆盒工具
- gazebo/world/urdf 配套调整

File: mm_description/urdf/mm_robot_gazebo.urdf.xacro (robot description, xacro)
@@ -29,5 +29,7 @@
          提供水平静摩擦约束. pad 居中, 平移时摩擦均匀, 不产生偏转; 静止时摩擦压住质心偏移
          引起的蠕动, 故车走直且静止不漂. 自转转速由 Nav2 controller/velocity_smoother 参数决定. -->
-    <!-- 居中贴地碰撞块: base_link 原点离地约 0.0476m, pad 厚 0.02m, 中心 z=-0.0376 使底面贴地 -->
+    <!-- 居中贴地承重板: base_link 原点离地约 0.0476m. 下移到 z=-0.0396 使板底略入地,
+         底盘改由这块宽板承重(轮子抬离约 1.6mm 变纯装饰), 板真正吃法向力 -> mu 才生效.
+         宽 0.18x0.18: 既给足摩擦压住漂移, 又提供支撑多边形防倾倒(小板承重会翻车). -->
     <link name="base_pad">
         <inertial>
@@ -38,5 +40,5 @@
             <origin xyz="0 0 0" rpy="0 0 0"/>
             <geometry>
-                <box size="0.03 0.03 0.02"/>
+                <box size="0.18 0.18 0.02"/>
             </geometry>
         </collision>
@@ -45,13 +47,23 @@
         <parent link="base_link"/>
         <child link="base_pad"/>
-        <origin xyz="0 0 -0.0376" rpy="0 0 0"/>
+        <origin xyz="0 0 -0.0396" rpy="0 0 0"/>
     </joint>
-    <!-- pad: 高摩擦但缩成中心小块(0.03x0.03). 抗漂移靠摩擦力 mu*N(与面积无关),
-         阻转靠摩擦力矩 ~mu*N*接触半径(与尺寸成正比). 大 pad(0.26)把自转力矩放大约30倍
-         压死转速; 缩到中心小块后抗漂移力不变, 阻转力矩趋近0 -> 既不漂又能原地自转.
-         防侧翻由四轮法向支撑保证(与 mu 无关). -->
+    <!-- pad 承重后 mu*N 才有意义: 高 mu 压住静止漂移. 驱动/自转时 planar_move 直接喂速度,
+         摩擦不阻止指令运动; 平板阻转力矩略增但可接受. 教训: 小块 pad 因不吃法向力(N≈0)
+         导致 mu 失效、底盘等于站冰面上漂移, 故改宽平板承重. -->
     <gazebo reference="base_pad">
-        <mu1>1.0</mu1>
-        <mu2>1.0</mu2>
+        <mu1>0.3</mu1>
+        <mu2>0.3</mu2>
+        <!-- 接触稳定 (治"平移+自转"组合工况平板弹跳/甩动 -> 导航乱飘, 及偏心质心引起的原地抖):
+             maxVel=0  穿透不注入 ODE 修正速度, 杀掉竖直弹跳;
+             minDepth  允许 2mm 微穿透给死区, 平板静置吃住法向力, mu*N 防漂保留;
+             kp 近刚性 + kd 重阻尼: 机械臂偏心质心压平板一边会激起小极限环(原地 buzz),
+             软弹簧(低kp)+轻阻尼会自激; 改高 kp 使边压不下去、大 kd 把振动能量耗掉.
+             目的: 底盘在全向组合指令下"运动==指令"且静止不抖, Nav2 参数针对理想运动学整定,
+             可直接移植真机(真机无此板, 靠真 Omni 轮). -->
+        <kp>1000000000000.0</kp>
+        <kd>1000.0</kd>
+        <minDepth>0.002</minDepth>
+        <maxVel>0.0</maxVel>
     </gazebo>
     <!-- 四轮零摩擦: 消除四角不对称切向力矩, 只保留视觉与法向支撑 -->
