Commit message: new arm

File: arm/arm_description/urdf/arm_description.urdf (robot description, URDF)
Before this commit: robot arm_description, 7 links, 6 joints
Joints:
- joint Joint_1: axis 0 0 1 -> 0 0 -1; limit lower=-2.4 upper=2.33 effort=10 velocity=1 -> lower=0 upper=4.712 effort=10 velocity=1; origin xyz=-0.00003461 0.04262805 0.07986836 rpy=0 0 0 -> xyz=-0.00003461 0.04262805 0.07986836 rpy=0 0 2.33001455
- joint Joint_2: axis 0 0 1 -> 0 0 -1; limit lower=-1.571 upper=0.524 effort=10 velocity=1 -> lower=0 upper=2.740 effort=10 velocity=1; origin xyz=0.0554 0 0.0663 rpy=0 1.57079633 0 -> xyz=0.0554 0 0.0663 rpy=1.57079633 0.40142573 1.57079633
- joint Joint_3: limit lower=-0.524 upper=1.571 effort=10 velocity=1 -> lower=0 upper=2.304 effort=10 velocity=1; origin xyz=-0.21500002 0 -0.0264 rpy=0 0 0 -> xyz=-0.21500002 0 -0.0264 rpy=0 0 -0.55850536
- joint Joint_4: axis 0 0 1 -> 0 0 -1; limit lower=-1.571 upper=1.571 effort=10 velocity=1 -> lower=0 upper=3.142 effort=10 velocity=1; origin xyz=0 0.04879037 -0.04004253 rpy=-3.14159265 1.56206849 -1.57079633 -> xyz=0 0.04879037 -0.04004253 rpy=1.57952416 0.00000000 3.14159265
- joint Joint_5: limit lower=0 upper=1.571 effort=10 velocity=1 -> lower=-1.571 upper=1.571 effort=10 velocity=1
